File: LEMSv2 PCB/LEMSv2.brd (EAGLE design)
At the start: 85.7 x 73.7 mm, 88 parts, among them J1 FEMALE 2x3, Q1 200mA/50V, Q10 200mA/50V, Q2 200mA/50V, Q3 MMBT3904, Q4 MMBT3904, Q5 200mA/50V, Q6 MMBT3904, Q7 200mA/50V, Q8 MMBT3904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

Commit message: Completed board
Parts:
- added U$4: MOUNTINGHOLE2.5, LEMSv2:MOUNTINGHOLE_2.5_PLATED
- FRAME1: value FRAME-LETTER -> FRAME-LETTERNO_PACKAGE; device SparkFun-Aesthetics:CREATIVE_COMMONS -> SparkFun-Aesthetics:DUMMY
- moved FRAME1 109.4 mm to (0.00, 0.00)
- moved R15 25.4 mm to (52.1, 55.6)
- moved LED1 24.8 mm to (56.5, 55.6), turned to 90 degrees
- moved R17 23.2 mm to (43.2, 55.6), turned to 0 degrees
- moved R16 21.4 mm to (52.1, 51.1)
- moved Q8 19.9 mm to (47.4, 55.6), turned to 270 degrees
- moved LED2 18.9 mm to (56.5, 51.1), turned to 90 degrees
- moved R18 14.4 mm to (43.2, 51.1), turned to 0 degrees
- moved Q9 13.5 mm to (47.4, 51.1), turned to 270 degrees
- moved BT1 2.44 mm to (6.60, 26.2)
Routing:
- net D7: track 0.00 -> 17.5 mm
- net GND: track 142.4 -> 154.9 mm, vias 9 -> 12
- net D6: track 0.00 -> 10.4 mm
- net N$7: track 0.00 -> 9.28 mm
- net N$8: track 0.00 -> 9.28 mm
- net 3.3V: track 27.3 -> 33.8 mm
- net VBAT_RTC: track 12.5 -> 16.9 mm
- net SDA: track 138.0 -> 141.9 mm
- net N$9: track 0.00 -> 3.79 mm
- net N$10: track 0.00 -> 3.79 mm
- net SCL: track 123.5 -> 126.3 mm
- net N$5: track 0.00 -> 2.57 mm
- net N$6: track 0.00 -> 2.57 mm
- net N$14: track 5.47 -> 8.01 mm
- net D5: track 37.3 -> 37.8 mm, vias 0 -> 1
Other:
- board text added: "+"
- board text added: "-"
- board text added: "3.3V"
- board text added: "5V"
- board text added: "AIN2"
- board text added: "AIN3"
- board text added: "CR1220"
- board text added: "FAN+"
- board text added: "FAN-"
- board text added: "GND"
- board text added: "L5TM DATA"
- board text added: "L5TM GND"
- board text added: "L5TM POW"
- board text added: "LEMSv2"
- board text added: "LI+"
- board text added: "LI-"
- board text added: "MISO"
- board text added: "MOSI"
- board text added: "NG"
- board text added: "OFF"
- board text added: "ON"
- board text added: "SCK"
- board text added: "SCL"
- board text added: "SCL 3.3V"
- board text added: "SCL 5V"
- board text added: "SDA"
- board text added: "SDA 3.3V"
- board text added: "SDA 5V"
- board text added: "SONIC DATA"
- board text added: "U5TM DATA"
- board text added: "U5TM GND"
- board text added: "U5TM POW"
- board text added: "University of Utah Environmental Fluid Dynamics"
- board text added: "VBAT"
- board text added: "WIND DIR"
- board text added: "WIND GND"
- board text added: "WIND POW"
- board text added: "WIND SPD"
- board text added: "x"
