File: LEMSv2 PCB/LEMSv2.brd (EAGLE design)
At the start: 85.7 x 73.7 mm, 89 parts, among them J1 FEMALE 2x3, Q1 200mA/50V, Q10 200mA/50V, Q2 200mA/50V, Q3 MMBT3904, Q4 MMBT3904, Q5 200mA/50V, Q6 MMBT3904, Q7 200mA/50V, Q8 MMBT3904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

Commit message: Added gerbers and centroid files
Parts:
- R12: value (none) -> 56k
- R22: value (none) -> 16k
Changed lines of the file:
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@@
 </class>
 </classes>
-<designrules name="LaenPCBOrder">
+<designrules name="OSHDesignRules">
 <description language="de">&lt;b&gt;EAGLE Design Rules&lt;/b&gt;
 &lt;p&gt;
@@
 <attribute name="VALUE" x="72.517" y="57.9756" size="0.4064" layer="27" ratio="10" rot="R90"/>
 </element>
-<element name="R12" library="LEMSv2" package="_0805" value="" x="69.088" y="3.81" locked="yes" smashed="yes" rot="R90">
+<element name="R12" library="LEMSv2" package="_0805" value="56k" x="69.088" y="3.81" locked="yes" smashed="yes" rot="R90">
 <attribute name="NAME" x="67.945" y="1.8415" size="0.8128" layer="25" ratio="18" rot="R90"/>
-<attribute name="VALUE" x="70.739" y="2.2226" size="0.4064" layer="27" ratio="10" rot="R90"/>
-</element>
-<element name="R22" library="LEMSv2" package="_0805" value="" x="65.786" y="3.81" locked="yes" smashed="yes" rot="R270">
+<attribute name="VALUE" x="69.6594" y="1.651" size="0.4064" layer="27" ratio="10" rot="R180"/>
+</element>
+<element name="R22" library="LEMSv2" package="_0805" value="16k" x="65.786" y="3.81" locked="yes" smashed="yes" rot="R270">
 <attribute name="NAME" x="63.881" y="4.1275" size="0.8128" layer="25" ratio="18" rot="R270"/>
-<attribute name="VALUE" x="64.135" y="5.3974" size="0.4064" layer="27" ratio="10" rot="R270"/>
+<attribute name="VALUE" x="65.3416" y="1.27" size="0.4064" layer="27" ratio="10"/>
 </element>
 <element name="R23" library="LEMSv2" package="_0805" value="75k" x="54.61" y="25.146"/>
