File: LEMSv2 PCB/LEMSv2.sch (EAGLE design)
At the start: 84 parts, among them J1 FEMALE 2x3, Q1 200mA/50V, Q10 200mA/50V, Q2 200mA/50V, Q3 MMBT3904, Q4 MMBT3904, Q5 200mA/50V, Q6 MMBT3904, Q7 200mA/50V, Q8 MMBT3904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

Commit message: More routing
Parts:
- added R12, R22: (no value), LEMSv2:RESISTOR_0805
- added R23, R24: 75k, LEMSv2:RESISTOR_0805
Connections:
- new net N$17: R23.2, U1.DAT1
- new net N$18: R24.2, U1.DAT2
- net 3.3V: now also R23.1, R24.1
- net A5: now also R12.2, R22.1
- net GND: now also R22.2
- net VBAT+: now also R12.1
Changed lines of the file:
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@@
 <part name="GND15" library="LEMSv2" deviceset="GND" device=""/>
 <part name="SUPPLY19" library="LEMSv2" deviceset="5V" device=""/>
+<part name="R12" library="LEMSv2" deviceset="RESISTOR" device="_0805"/>
+<part name="R22" library="LEMSv2" deviceset="RESISTOR" device="_0805"/>
+<part name="GND16" library="LEMSv2" deviceset="GND" device=""/>
+<part name="R23" library="LEMSv2" deviceset="RESISTOR" device="_0805" value="75k"/>
+<part name="R24" library="LEMSv2" deviceset="RESISTOR" device="_0805" value="75k"/>
+<part name="SUPPLY20" library="LEMSv2" deviceset="3.3V" device=""/>
 </parts>
 <sheets>
@@
 <instance part="GND15" gate="1" x="121.92" y="111.76"/>
 <instance part="SUPPLY19" gate="G$1" x="121.92" y="132.08"/>
+<instance part="R12" gate="G$1" x="220.98" y="43.18"/>
+<instance part="R22" gate="G$1" x="233.68" y="43.18"/>
+<instance part="GND16" gate="1" x="241.3" y="40.64"/>
+<instance part="R23" gate="G$1" x="231.14" y="127"/>
+<instance part="R24" gate="G$1" x="231.14" y="121.92"/>
+<instance part="SUPPLY20" gate="G$1" x="223.52" y="127"/>
 </instances>
 <busses>
@@
 <wire x1="53.34" y1="88.9" x2="58.42" y2="88.9" width="0.1524" layer="91"/>
 <label x="53.34" y="88.9" size="1.778" layer="95"/>
+</segment>
+<segment>
+<pinref part="R24" gate="G$1" pin="1"/>
+<pinref part="R23" gate="G$1" pin="1"/>
+<wire x1="226.06" y1="121.92" x2="226.06" y2="127" width="0.1524" layer="91"/>
+<pinref part="SUPPLY20" gate="G$1" pin="3.3V"/>
+<wire x1="223.52" y1="127" x2="226.06" y2="127" width="0.1524" layer="91"/>
+<junction x="226.06" y="127"/>
 </segment>
 </net>
@@
 <pinref part="GND15" gate="1" pin="GND"/>
 </segment>
+<segment>
+<pinref part="R22" gate="G$1" pin="2"/>
+<pinref part="GND16" gate="1" pin="GND"/>
+<wire x1="238.76" y1="43.18" x2="241.3" y2="43.18" width="0.1524" layer="91"/>
+</segment>
 </net>
 <net name="SCK" class="0">
@@
 <pinref part="U1" gate="G$1" pin="SCLK"/>
 <wire x1="233.68" y1="149.86" x2="238.76" y2="149.86" width="0.1524" layer="91"/>
-<label x="236.22" y="149.86" size="1.778" layer="95"/>
+<label x="233.68" y="149.86" size="1.778" layer="95"/>
 </segment>
 <segment>
@@
 <pinref part="U1" gate="G$1" pin="DATA_IN"/>
 <wire x1="233.68" y1="147.32" x2="238.76" y2="147.32" width="0.1524" layer="91"/>
-<label x="236.22" y="147.32" size="1.778" layer="95"/>
+<label x="233.68" y="147.32" size="1.778" layer="95"/>
 </segment>
 <segment>
@@
 <pinref part="U1" gate="G$1" pin="DATA_OUT"/>
 <wire x1="233.68" y1="144.78" x2="238.76" y2="144.78" width="0.1524" layer="91"/>
-<label x="236.22" y="144.78" size="1.778" layer="95"/>
+<label x="233.68" y="144.78" size="1.778" layer="95"/>
 </segment>
 <segment>
@@
 <pinref part="U1" gate="G$1" pin="CS"/>
 <wire x1="233.68" y1="152.4" x2="238.76" y2="152.4" width="0.1524" layer="91"/>
-<label x="236.22" y="152.4" size="1.778" layer="95"/>
+<label x="233.68" y="152.4" size="1.778" layer="95"/>
 </segment>
 <segment>
@@
 <wire x1="137.16" y1="127" x2="132.08" y2="127" width="0.1524" layer="91"/>
 <label x="132.08" y="127" size="1.778" layer="95"/>
+</segment>
+<segment>
+<pinref part="R12" gate="G$1" pin="2"/>
+<pinref part="R22" gate="G$1" pin="1"/>
+<wire x1="226.06" y1="43.18" x2="228.6" y2="43.18" width="0.1524" layer="91"/>
+<wire x1="228.6" y1="43.18" x2="228.6" y2="38.1" width="0.1524" layer="91"/>
+<junction x="228.6" y="43.18"/>
+<label x="228.6" y="38.1" size="1.778" layer="95" rot="R90"/>
 </segment>
 </net>
@@
 <wire x1="213.36" y1="48.26" x2="223.52" y2="48.26" width="0.1524" layer="91"/>
 <label x="215.9" y="48.26" size="1.778" layer="95"/>
+<pinref part="R12" gate="G$1" pin="1"/>
+<wire x1="215.9" y1="43.18" x2="213.36" y2="43.18" width="0.1524" layer="91"/>
+<wire x1="213.36" y1="43.18" x2="213.36" y2="48.26" width="0.1524" layer="91"/>
+<junction x="213.36" y="48.26"/>
 </segment>
 </net>
@@
 </segment>
 </net>
+<net name="N$17" class="0">
+<segment>
+<pinref part="R23" gate="G$1" pin="2"/>
+<wire x1="236.22" y1="127" x2="243.84" y2="127" width="0.1524" layer="91"/>
+<wire x1="243.84" y1="127" x2="243.84" y2="154.94" width="0.1524" layer="91"/>
+<pinref part="U1" gate="G$1" pin="DAT1"/>
+<wire x1="243.84" y1="154.94" x2="233.68" y2="154.94" width="0.1524" layer="91"/>
+</segment>
+</net>
+<net name="N$18" class="0">
+<segment>
+<pinref part="U1" gate="G$1" pin="DAT2"/>
+<wire x1="233.68" y1="157.48" x2="246.38" y2="157.48" width="0.1524" layer="91"/>
+<wire x1="246.38" y1="157.48" x2="246.38" y2="121.92" width="0.1524" layer="91"/>
+<pinref part="R24" gate="G$1" pin="2"/>
+<wire x1="246.38" y1="121.92" x2="236.22" y2="121.92" width="0.1524" layer="91"/>
+</segment>
+</net>

Commit message: Completed board
Parts:
- added U$4: MOUNTINGHOLE2.5, LEMSv2:MOUNTINGHOLE2.5
- FRAME1: value FRAME-LETTER -> FRAME-LETTERNO_PACKAGE; device SparkFun-Aesthetics:FRAME-LETTER -> SparkFun-Aesthetics:FRAME-LETTERNO_PACKAGE
Changed lines of the file:
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@@
 </classes>
 <parts>
-<part name="FRAME1" library="SparkFun-Aesthetics" deviceset="FRAME-LETTER" device=""/>
+<part name="FRAME1" library="SparkFun-Aesthetics" deviceset="FRAME-LETTER" device="NO_PACKAGE" value="FRAME-LETTERNO_PACKAGE"/>
 <part name="U1" library="LEMSv2" deviceset="SDMMC" device="06132"/>
 <part name="GND2" library="LEMSv2" deviceset="GND" device=""/>
@@
 <part name="R24" library="LEMSv2" deviceset="RESISTOR" device="_0805" value="75k"/>
 <part name="SUPPLY20" library="LEMSv2" deviceset="3.3V" device=""/>
+<part name="U$4" library="LEMSv2" deviceset="MOUNTINGHOLE" device="2.5"/>
 </parts>
 <sheets>
@@
 <instance part="R24" gate="G$1" x="231.14" y="121.92"/>
 <instance part="SUPPLY20" gate="G$1" x="223.52" y="127"/>
+<instance part="U$4" gate="G$1" x="187.96" y="43.18"/>
 </instances>
 <busses>
